File: cm4-carrier-net.kicad_sch (KiCad schematic)
At the start: 68 parts, among them J1 USB_C_Receptacle_USB2.0, J2 Micro_SD_Card, J3 Abracon_ARJM11-502, J4 20021121-00010C4LF, J5 block, J6 USB_A, Q1 DMP2066LSN, Q2 FDMT800152DC, Q3 FDMT800152DC, SW1 BOOT, SW2 GLOBAL_EN, SW4 USB_OTG, U1 TPS54302, U2 LTC4365TS8, U3 ORANGE_PI_CM4, U6 TPD2EUSB30

Commit message: added thingies
began creating daughter board and added stm32 for led control
Parts:
- added U4: STM32C011J4Mx, Package_DFN_QFN:ST_UFQFPN-20_3x3mm_P0.5mm, symbol MCU_ST_STM32C0:STM32C011J4Mx
Connections:
- net +3.3V: now also J4.8, U4.2 (VDD)
- net GND: now also U4.3 (VSS)
- net I2C1_SCL-: now also U4.1 (PC14/PB7); no longer J4.5
- net I2C1_SDA+: now also U4.4 (PF2/PA0/PA1/PA2); no longer J4.3
- net I2C_TO_DB_SDA: now reaches J4.7
- net I2C_TO_DB_SDA: now also U4.5 (PA8/PA9/PA11)
- new net I2C_TO_DB_SCL: J4.5, U4.6 (PA10/PA12)
- new net LED_DRIVER_RST: J4.3, U4.7 (PA13)
Changed lines of the file:
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@@
     (effects (font (size 1.27 1.27)) (justify left bottom))
   )
-  (label "I2C1_SDA+" (at 521.97 72.39 180) (fields_autoplaced)
-    (effects (font (size 1.27 1.27)) (justify right bottom))
-  )
   (label "E0_TR1-" (at 67.31 133.35 0) (fields_autoplaced)
     (effects (font (size 1.27 1.27)) (justify left bottom))
@@
     (effects (font (size 1.27 1.27)) (justify right bottom))
   )
+  (label "I2C_TO_DB_SDA" (at 521.97 77.47 180) (fields_autoplaced)
+    (effects (font (size 1.27 1.27)) (justify right bottom))
+  )
   (label "E0_TR2+" (at 67.31 128.27 0) (fields_autoplaced)
     (effects (font (size 1.27 1.27)) (justify left bottom))
@@
     (effects (font (size 1.27 1.27)) (justify left bottom))
   )
+  (label "I2C1_SCL-" (at 500.38 100.33 180) (fields_autoplaced)
+    (effects (font (size 1.27 1.27)) (justify right bottom))
+  )
+  (label "LED_DRIVER_RST" (at 543.56 100.33 0) (fields_autoplaced)
+    (effects (font (size 1.27 1.27)) (justify left bottom))
+  )
   (label "PI_LED_nACT" (at 309.88 53.34 180) (fields_autoplaced)
     (effects (font (size 1.27 1.27)) (justify right bottom))
@@
     (effects (font (size 1.27 1.27)) (justify right bottom))
   )
-  (label "I2C1_SCL-" (at 521.97 74.93 180) (fields_autoplaced)
+  (label "I2C_TO_DB_SCL" (at 521.97 74.93 180) (fields_autoplaced)
     (effects (font (size 1.27 1.27)) (justify right bottom))
   )
+  (label "I2C_TO_DB_SDA" (at 543.56 95.25 0) (fields_autoplaced)
+    (effects (font (size 1.27 1.27)) (justify left bottom))
+  )
   (label "E0_TR2-" (at 67.31 125.73 0) (fields_autoplaced)
     (effects (font (size 1.27 1.27)) (justify left bottom))
@@
     (effects (font (size 1.27 1.27)) (justify right bottom))
   )
+  (label "I2C1_SDA+" (at 500.38 95.25 180) (fields_autoplaced)
+    (effects (font (size 1.27 1.27)) (justify right bottom))
+  )
   (label "USB1-" (at 492.76 30.48 180) (fields_autoplaced)
     (effects (font (size 1.27 1.27)) (justify right bottom))
@@
     (effects (font (size 1.27 1.27)) (justify right bottom))
   )
+  (label "LED_DRIVER_RST" (at 521.97 72.39 180) (fields_autoplaced)
+    (effects (font (size 1.27 1.27)) (justify right bottom))
+  )
   (label "E0_TR0+" (at 386.08 40.64 0) (fields_autoplaced)
     (effects (font (size 1.27 1.27)) (justify left bottom))
@@
     (effects (font (size 1.27 1.27)) (justify left bottom))
   )
+  (label "I2C_TO_DB_SCL" (at 543.56 97.79 0) (fields_autoplaced)
+    (effects (font (size 1.27 1.27)) (justify left bottom))
+  )
   (label "SD_PWR" (at 160.02 176.53 0) (fields_autoplaced)
     (effects (font (size 1.27 1.27)) (justify left bottom))
@@
     )
   )
+  (symbol (lib_id "power:GND") (at 523.24 110.49 0) (unit 1)
+    (in_bom yes) (on_board yes) (dnp no) (fields_autoplaced)
+    (property "Reference" "#PWR033" (at 523.24 116.84 0)
+      (effects (font (size 1.27 1.27)) hide)
+    )
+    (property "Value" "GND" (at 523.24 115.57 0)
+      (effects (font (size 1.27 1.27)))
+    )
+    (property "Footprint" "" (at 523.24 110.49 0)
+      (effects (font (size 1.27 1.27)) hide)
+    )
+    (property "Datasheet" "" (at 523.24 110.49 0)
+      (effects (font (size 1.27 1.27)) hide)
+    )
+    (pin "1")
+    (instances
+      (project "cm4-carrier-net"
+        (path "/a58a5c23-cf42-4abb-bf4c-19a657300252"
+          (reference "#PWR033") (unit 1)
+        )
+      )
+    )
+  )
   (symbol (lib_id "Device:C") (at 264.16 132.08 0) (unit 1)
     (in_bom yes) (on_board yes) (dnp no)
@@
     )
   )
+  (symbol (lib_id "power:+3.3V") (at 523.24 90.17 0) (unit 1)
+    (in_bom yes) (on_board yes) (dnp no)
+    (property "Reference" "#PWR032" (at 523.24 93.98 0)
+      (effects (font (size 1.27 1.27)) hide)
+    )
+    (property "Value" "+3.3V" (at 523.24 86.36 0)
+      (effects (font (size 1.27 1.27)))
+    )
+    (property "Footprint" "" (at 523.24 90.17 0)
+      (effects (font (size 1.27 1.27)) hide)
+    )
+    (property "Datasheet" "" (at 523.24 90.17 0)
+      (effects (font (size 1.27 1.27)) hide)
+    )
+    (pin "1")
+    (instances
+      (project "cm4-carrier-net"
+        (path "/a58a5c23-cf42-4abb-bf4c-19a657300252"
+          (reference "#PWR032") (unit 1)
+        )
+      )
+    )
+  )
+  (symbol (lib_id "MCU_ST_STM32C0:STM32C011J4Mx") (at 520.7 100.33 0) (unit 1)
+    (in_bom yes) (on_board yes) (dnp no) (fields_autoplaced)
+    (property "Reference" "U4" (at 525.4341 87.63 0)
+      (effects (font (size 1.27 1.27)) (justify left))
+    )
+    (property "Value" "STM32C011J4Mx" (at 525.4341 90.17 0)
+      (effects (font (size 1.27 1.27)) (justify left))
+    )
+    (property "Footprint" "Package_DFN_QFN:ST_UFQFPN-20_3x3mm_P0.5mm" (at 502.92 107.95 0)
+      (effects (font (size 1.27 1.27)) (justify right) hide)
+    )
+    (property "Datasheet" "https://www.st.com/resource/en/datasheet/stm32c011j4.pdf" (at 520.7 100.33 0)
+      (effects (font (size 1.27 1.27)) hide)
+    )
+    (pin "5")
+    (pin "3")
+    (pin "2")
+    (pin "1")
+    (pin "8")
+    (pin "4")
+    (pin "6")
+    (pin "7")
+    (instances
+      (project "cm4-carrier-net"
+        (path "/a58a5c23-cf42-4abb-bf4c-19a657300252"
+          (reference "U4") (unit 1)
+        )
+      )
+    )
+  )
   (symbol (lib_id "Device:R_Small_US") (at 179.07 160.02 0) (unit 1)
     (in_bom yes) (on_board yes) (dnp no)
@@
         )
       )
+    )
+  )
+  (symbol (lib_id "power:+3.3V") (at 532.13 77.47 270) (unit 1)
+    (in_bom yes) (on_board yes) (dnp no)
+    (property "Reference" "#PWR031" (at 528.32 77.47 0)
+      (effects (font (size 1.27 1.27)) hide)
+    )
+    (property "Value" "+3.3V" (at 535.94 77.47 0)
+      (effects (font (size 1.27 1.27)))
+    )
+    (property "Footprint" "" (at 532.13 77.47 0)
+      (effects (font (size 1.27 1.27)) hide)
+    )
+    (property "Datasheet" "" (at 532.13 77.47 0)
+      (effects (font (size 1.27 1.27)) hide)
+    )
+    (pin "1")
+    (instances
+      (project "cm4-carrier-net"
+        (path "/a58a5c23-cf42-4abb-bf4c-19a657300252"
+          (reference "#PWR031") (unit 1)
+        )
+      )

Commit message: added some things
Parts:
- added J7: 20021121-00010C4LF, digikey-footprints:PinHeader_2x5_P1.27mm, symbol dk_Rectangular-Connectors-Headers-Male-Pins:20021121-00010C4LF
Connections:
- net CAMERA_PDN: now reaches U3.JP1_97 (CAMERA_PDN_L)
- net MIPI_CSI_RX0_D0N: now reaches U3.JP2_15 (MIPI_CSI_RX0_D0N)
- net MIPI_CSI_RX0_D0P: now reaches U3.JP2_17 (MIPI_CSI_RX0_D0P)
- net MIPI_CSI_RX1_D0N: now reaches U3.JP2_21 (MIPI_CSI_RX0_D1N)
- net MIPI_CSI_RX1_D0P: now reaches U3.JP2_23 (MIPI_CSI_RX0_D1P)
- net MIPI_CSI_RX_CLK0N: now reaches U3.JP2_27 (MIPI_CSI_RX_CLK0N)
- net MIPI_CSI_RX_CLK0P: now reaches U3.JP2_29 (MIPI_CSI_RX_CLK0P)
Other:
- moved on the sheet: J4
