File: _autosave-cm4-carrier-net.kicad_sch (KiCad schematic)
At the start: 69 parts, among them J1 USB_C_Receptacle_USB2.0, J2 Conn_01x15_MountingPin, J2 Micro_SD_Card, J3 Abracon_ARJM11-502, J4 20021121-00010C4LF, J5 block, J6 USB_A, Q1 DMP2066LSN, Q2 FDMT800152DC, Q3 FDMT800152DC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

Commit message: added camera zif connector
Parts:
- removed J4: 20021121-00010C4LF, digikey-footprints:PinHeader_2x5_P1.27mm, symbol dk_Rectangular-Connectors-Headers-Male-Pins:20021121-00010C4LF
Changed lines of the file:
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@@
-    )
-  )
-  (symbol (lib_id "power:GND") (at 533.4 80.01 270) (unit 1)
-    (in_bom yes) (on_board yes) (dnp no) (fields_autoplaced)
-    (property "Reference" "#PWR023" (at 527.05 80.01 0)
-      (effects (font (size 1.27 1.27)) hide)
-    )
-    (property "Value" "GND" (at 529.59 80.01 90)
-      (effects (font (size 1.27 1.27)) (justify right))
-    )
-    (property "Footprint" "" (at 533.4 80.01 0)
-      (effects (font (size 1.27 1.27)) hide)
-    )
-    (property "Datasheet" "" (at 533.4 80.01 0)
-      (effects (font (size 1.27 1.27)) hide)
-    )
-    (pin "1")
-    (instances
-      (project "cm4-carrier-net"
-        (path "/a58a5c23-cf42-4abb-bf4c-19a657300252"
-          (reference "#PWR023") (unit 1)
-        )
-      )
     )
   )
@@
     )
   )
-  (symbol (lib_id "power:+5V") (at 533.4 69.85 90) (unit 1)
-    (in_bom yes) (on_board yes) (dnp no)
-    (property "Reference" "#PWR022" (at 537.21 69.85 0)
-      (effects (font (size 1.27 1.27)) hide)
-    )
-    (property "Value" "+5V" (at 529.59 68.58 0)
-      (effects (font (size 1.27 1.27)))
-    )
-    (property "Footprint" "" (at 533.4 69.85 0)
-      (effects (font (size 1.27 1.27)) hide)
-    )
-    (property "Datasheet" "" (at 533.4 69.85 0)
-      (effects (font (size 1.27 1.27)) hide)
-    )
-    (pin "1")
-    (instances
-      (project "cm4-carrier-net"
-        (path "/a58a5c23-cf42-4abb-bf4c-19a657300252"
-          (reference "#PWR022") (unit 1)
-        )
-      )
-    )
-  )
   (symbol (lib_id "power:GND") (at 495.3 85.09 0) (unit 1)
     (in_bom yes) (on_board yes) (dnp no) (fields_autoplaced)
@@
     )
   )
-  (symbol (lib_id "dk_Rectangular-Connectors-Headers-Male-Pins:20021121-00010C4LF") (at 538.48 74.93 0) (unit 1)
-    (in_bom yes) (on_board yes) (dnp no) (fields_autoplaced)
-    (property "Reference" "J4" (at 538.48 63.5 0)
-      (effects (font (size 1.27 1.27)))
-    )
-    (property "Value" "20021121-00010C4LF" (at 538.48 66.04 0)
-      (effects (font (size 1.27 1.27)))
-    )
-    (property "Footprint" "digikey-footprints:PinHeader_2x5_P1.27mm" (at 543.56 69.85 0)
-      (effects (font (size 1.524 1.524)) (justify left) hide)
-    )
-    (property "Datasheet" "https://cdn.amphenol-icc.com/media/wysiwyg/files/drawing/20021121.pdf" (at 543.56 67.31 0)
-      (effects (font (size 1.524 1.524)) (justify left) hide)
-    )
-    (property "Digi-Key_PN" "609-3695-1-ND" (at 543.56 64.77 0)
-      (effects (font (size 1.524 1.524)) (justify left) hide)
-    )
-    (property "MPN" "20021121-00010C4LF" (at 543.56 62.23 0)
-      (effects (font (size 1.524 1.524)) (justify left) hide)
-    )
-    (property "Category" "Connectors, Interconnects" (at 543.56 59.69 0)
-      (effects (font (size 1.524 1.524)) (justify left) hide)
-    )
-    (property "Family" "Rectangular Connectors - Headers, Male Pins" (at 543.56 57.15 0)
-      (effects (font (size 1.524 1.524)) (justify left) hide)
-    )
-    (property "DK_Datasheet_Link" "https://cdn.amphenol-icc.com/media/wysiwyg/files/drawing/20021121.pdf" (at 543.56 54.61 0)
-      (effects (font (size 1.524 1.524)) (justify left) hide)
-    )
-    (property "DK_Detail_Page" "/product-detail/en/amphenol-icc-fci/20021121-00010C4LF/609-3695-1-ND/2209147" (at 543.56 52.07 0)
-      (effects (font (size 1.524 1.524)) (justify left) hide)
-    )
-    (property "Description" "CONN HEADER SMD 10POS 1.27MM" (at 543.56 49.53 0)
-      (effects (font (size 1.524 1.524)) (justify left) hide)
-    )
-    (property "Manufacturer" "Amphenol ICC (FCI)" (at 543.56 46.99 0)
-      (effects (font (size 1.524 1.524)) (justify left) hide)
-    )
-    (property "Status" "Active" (at 543.56 44.45 0)
-      (effects (font (size 1.524 1.524)) (justify left) hide)
-    )
-    (pin "1")
-    (pin "10")
-    (pin "2")
-    (pin "3")
-    (pin "4")
-    (pin "5")
-    (pin "6")
-    (pin "7")
-    (pin "8")
-    (pin "9")
-    (instances
-      (project "cm4-carrier-net"
-        (path "/a58a5c23-cf42-4abb-bf4c-19a657300252"
-          (reference "J4") (unit 1)
-        )
-      )
-    )
-  )
   (symbol (lib_id "Device:R_Small_US") (at 205.74 134.62 0) (unit 1)
     (in_bom yes) (on_board yes) (dnp no)
@@
         )
       )
-    )
-  )
-  (symbol (lib_id "power:+5V") (at 543.56 69.85 270) (unit 1)
-    (in_bom yes) (on_board yes) (dnp no)
-    (property "Reference" "#PWR024" (at 539.75 69.85 0)
-      (effects (font (size 1.27 1.27)) hide)
-    )
-    (property "Value" "+5V" (at 547.37 68.58 0)
-      (effects (font (size 1.27 1.27)))
-    )
-    (property "Footprint" "" (at 543.56 69.85 0)
-      (effects (font (size 1.27 1.27)) hide)
-    )
-    (property "Datasheet" "" (at 543.56 69.85 0)
-      (effects (font (size 1.27 1.27)) hide)
-    )
-    (pin "1")
-    (instances
-      (project "cm4-carrier-net"
-        (path "/a58a5c23-cf42-4abb-bf4c-19a657300252"
-          (reference "#PWR024") (unit 1)
-        )
-      )
-    )
-  )
-  (symbol (lib_id "power:GND") (at 543.56 80.01 90) (unit 1)
-    (in_bom yes) (on_board yes) (dnp no) (fields_autoplaced)
-    (property "Reference" "#PWR030" (at 549.91 80.01 0)
-      (effects (font (size 1.27 1.27)) hide)
-    )
-    (property "Value" "GND" (at 547.37 80.01 90)
-      (effects (font (size 1.27 1.27)) (justify right))
-    )
-    (property "Footprint" "" (at 543.56 80.01 0)
-      (effects (font (size 1.27 1.27)) hide)
-    )
-    (property "Datasheet" "" (at 543.56 80.01 0)
-      (effects (font (size 1.27 1.27)) hide)
-    )
-    (pin "1")
-    (instances
-      (project "cm4-carrier-net"
-        (path "/a58a5c23-cf42-4abb-bf4c-19a657300252"
-          (reference "#PWR030") (unit 1)
-        )
-      )
