File: _autosave-cm4-carrier-net.kicad_sch (KiCad schematic)
At the start: 70 parts, among them J1 USB_C_Receptacle_USB2.0, J2 Conn_01x15_MountingPin, J3 54602-908LF, J5 block, J6 USB_A, M1 Fan, Q2 LTC4412ES6_TRMPBF, Q3 IRLML6401TRPBF, Q4 IRLML6401TRPBF, SW1 BOOT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

Commit message: google coral tpu
Parts:
- removed C16: 47uF, Capacitor_SMD:C_1206_3216Metric, symbol Device:C
Connections:
- net +1V8: now also U2.83 (USB_SEL)
- net GND: now also U2.10 (PCIE_REFCLK_N), U2.11 (PCIE_REFCLK_P), U2.7 (PCIE_RX_P), U2.8 (PCIE_RX_N)
- net PCIE_TX_N: no longer U2.4 (PCIE_TX_N), U3.JP2_24 (PCIE20_TXN)
- net PCIE_TX_P: no longer U2.5 (PCIE_TX_P), U3.JP2_22 (PCIE20_TXP)
- net USB_CORAL-: now reaches U3.JP3_19 (USB3_HOST1_DM)
- net USB_CORAL-: now also U2.14 (USB2_D_N)
- net USB_CORAL+: now reaches U3.JP3_21 (USB3_HOST1_DP)
- net USB_CORAL+: now also U2.13 (USB2_D_P)
- net PCIE_REFCLK_N: no longer names the net of U3.JP2_10 (PCIE20_REFCLKP_P)
- net PCIE_REFCLK_N: no longer U2.10 (PCIE_REFCLK_N)
- net PCIE_REFCLK_P: no longer names the net of U3.JP2_12 (PCIE20_REFCLKP_N)
- net PCIE_REFCLK_P: no longer U2.11 (PCIE_REFCLK_P)
- net PCIE_RX_N: no longer names the net of U3.JP2_18 (PCIE20_RXN)
- net PCIE_RX_N: no longer U2.8 (PCIE_RX_N)
- net PCIE_RX_P: no longer names the net of U3.JP2_16 (PCIE20_RXP)
- net PCIE_RX_P: no longer U2.7 (PCIE_RX_P)
- no-connect marks 3 -> 8
