File: cm4-carrier-net.kicad_pcb (KiCad board)
At the start: 4 copper layers, 91.6 x 50.4 mm, 68 parts, among them J1 USB_C_Receptacle_USB2.0, J2 Micro_SD_Card, J3 Abracon_ARJM11-502, J5 block, J6 USB_A, J8 Conn_01x15_MountingPin, Q1 DMP2066LSN, Q2 FDMT800152DC, Q3 FDMT800152DC, SW1 BOOT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

Commit message: cleaned up pcb routing
Routing:
- net /CAMERA_PDN: track 61.5 -> 0.00 mm, vias 4 -> 0

Commit message: cleaned up the pcb a little bit
Parts:
- moved H1 10.5 mm to (83.5, 87.0)
- moved H3 10.5 mm to (166.5, 87.0)
- moved J6 10.4 mm to (95.5, 89.9)
- moved J1 10.3 mm to (95.5, 88.0)
- moved C5 4.34 mm to (99.8, 93.5), turned to -90 degrees
Routing:
- net /I2C1_SCL-: track 0.00 -> 79.8 mm
- net /I2C1_SDA+: track 0.00 -> 75.3 mm, vias 0 -> 2
- net /CAMERA_PDN: track 0.00 -> 74.1 mm
- net +3.3V: track 159.5 -> 207.3 mm, vias 0 -> 2
- net /SD_PWR: track 54.2 -> 71.9 mm
- net Net-(J1-SHIELD): track 2.10 -> 19.6 mm
- net GND: track 157.0 -> 173.0 mm
- net /USB_D+: track 51.6 -> 62.7 mm
- net /USB_D-: track 55.3 -> 66.3 mm
- net /USB+: track 22.5 -> 33.3 mm
- net /USB-: track 22.8 -> 33.2 mm
- net Net-(J1-CC1): track 3.11 -> 13.3 mm
- net Net-(J1-CC2): track 2.57 -> 12.7 mm
- net /USB_VBUS: track 13.5 -> 19.0 mm
- net +5V: track 138.1 -> 134.1 mm, vias 5 -> 4
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Other:
- board size 91.6 x 50.4 mm -> 91.4 x 50.4 mm
