File: _autosave-cm4-carrier-net.kicad_pcb (KiCad board)
At the start: 4 copper layers, 91.4 x 56.5 mm, 69 parts, among them J1 USB_C_Receptacle_USB2.0, J3 54602-908LF, J5 block, J6 USB_A, J8 Conn_01x15_MountingPin, M1 Fan, Q2 LTC4412ES6_TRMPBF, Q3 IRLML6401TRPBF, Q4 IRLML6401TRPBF, SW1 BOOT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

Commit message: google coral tpu
Routing:
- net GND: track 83.8 -> 158.0 mm, vias 112 -> 144
- net /USB_OTG_ID: track 0.00 -> 36.1 mm, vias 0 -> 1
